File: kicad/juniper-1/juniper-1.kicad_pcb (KiCad board)
At the start: 4 copper layers, 53 parts, among them J1 BOOT_OPTION, J2 UART, J3 ENCODER, J4 BATT_INPUT, J5 1714984, Q1 NTMFS5C645NL, Q2 NTMFS5C645NL, Q3 NTMFS5C645NL, Q4 NTMFS5C645NL, Q5 NTMFS5C645NL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

Commit message: made lots of progress with rerouting the PCB
Parts:
- J4: footprint Connector_AMASS:AMASS_XT60-F_1x02_P7.20mm_Vertical -> Connector_AMASS:AMASS_XT60-M_1x02_P7.20mm_Vertical
- moved C19 102.0 mm to (182.5, 92.0), turned to 180 degrees
- moved C20 91.5 mm to (182.5, 83.0), turned to 180 degrees
- moved SW1 90.3 mm to (165.0, 110.0)
- moved C16 66.8 mm to (154.0, 115.5), turned to 90 degrees
- moved C1 60.2 mm to (122.5, 124.8), turned to 90 degrees
- moved C2 59.8 mm to (135.5, 124.8), turned to 90 degrees
- moved C3 59.4 mm to (148.5, 124.8), turned to 90 degrees
- moved C4 59.1 mm to (161.5, 124.8), turned to 90 degrees
- moved R4 54.4 mm to (175.0, 78.0), turned to 0 degrees
- moved J2 53.9 mm to (144.5, 73.5), turned to 0 degrees
- moved U4 52.0 mm to (150.0, 112.0), turned to 0 degrees
- moved R12 49.9 mm to (127.1, 115.0)
- moved R9 48.1 mm to (175.0, 85.5), turned to 0 degrees
- moved U1 47.1 mm to (137.0, 78.5), turned to 0 degrees
- moved R14 42.4 mm to (175.0, 93.0), turned to 0 degrees
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Routing:
- net VMO-: track 150.2 -> 66.3 mm, vias 4 -> 5
- net EN: track 93.8 -> 17.2 mm, vias 0 -> 3
- net RXD0: track 90.1 -> 37.8 mm, vias 0 -> 2
- net IO7: track 3.90 -> 54.4 mm, vias 0 -> 2
- net TXD0: track 86.1 -> 36.9 mm, vias 0 -> 2
- net Net-(C9-Pad2): track 0.00 -> 49.0 mm, vias 0 -> 2
- net CU: track 0.00 -> 38.6 mm, vias 0 -> 2
- net IO8: track 9.92 -> 47.6 mm, vias 0 -> 2
- net 12VOUT: track 0.00 -> 37.1 mm, vias 0 -> 2
- net IO1: track 10.5 -> 44.8 mm
- net LSW: track 0.00 -> 30.3 mm, vias 0 -> 2
- net IO0: track 51.6 -> 21.7 mm
- net IO2: track 12.6 -> 42.2 mm
- net LSV: track 0.00 -> 28.1 mm, vias 0 -> 2
- net IO3: track 12.4 -> 40.2 mm
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- removed copper zone on In2.Cu, net VMO+
